File: hw/Luminography.kicad_pcb (KiCad board)
At the start: 2 copper layers, 100 x 100 mm, 110 parts, among them J1 USB_C_Receptacle_PowerOnly_6P, J2 Conn_01x04, Q1 2N7002, SW1 SW_Push, SW2 SW_Push, U1 LTC4054ES5-4.2, U10 MAX98357AETE+, U100 BH1750FVI-TR, U101 BH1750FVI-TR, U102 BH1750FVI-TR, U103 BH1750FVI-TR, U104 BH1750FVI-TR, U105 BH1750FVI-TR, U106 BH1750FVI-TR, U107 BH1750FVI-TR, U108 BH1750FVI-TR, U109 BH1750FVI-TR, U110 BH1750FVI-TR, U111 BH1750FVI-TR, U112 BH1750FVI-TR, U113 BH1750FVI-TR, U114 BH1750FVI-TR, U115 BH1750FVI-TR, U116 BH1750FVI-TR, U117 BH1750FVI-TR, U118 BH1750FVI-TR, U119 BH1750FVI-TR, U120 BH1750FVI-TR, U121 BH1750FVI-TR, U122 BH1750FVI-TR, U123 BH1750FVI-TR, U2 XS3A1T3157GMX, U3 SPX3819M5-L-3-3, U4 MAX17048G+T10, U5 STM32G030K6Tx, U6 ZJY128R-IG01, U7 W25Q16JVUXIQ, U8 BMI270, U9 MMC5603NJ, X1 12.288MHz

Commit message: Board design almost done, do later
Connections:
- U5 pad 10: I2Cx_SDA_03 -> I2Cx_SDA_08
- U5 pad 11: I2Cx_SDA_04 -> I2Cx_SDA_09
- U5 pad 12: I2Cx_SDA_05 -> I2Cx_SDA_10
- U5 pad 13: I2Cx_SDA_06 -> I2Cx_SDA_11
- U5 pad 14: I2Cx_SDA_07 -> I2Cx_SDA_00
- U5 pad 15: I2Cx_SDA_08 -> I2Cx_SDA_01
- U5 pad 16: I2Cx_SDA_09 -> I2Cx_SDA_02
- U5 pad 17: I2Cx_SDA_10 -> I2Cx_SDA_03
- U5 pad 18: I2Cx_SDA_11 -> I2Cx_SDA_04
- U5 pad 7: I2Cx_SDA_00 -> I2Cx_SDA_05
- U5 pad 8: I2Cx_SDA_01 -> I2Cx_SDA_06
- U5 pad 9: I2Cx_SDA_02 -> I2Cx_SDA_07
Routing:
- net I2Cx_SDA_04: track 13.9 -> 110.4 mm
- net I2Cx_SDA_03: track 13.9 -> 91.6 mm
- net I2Cx_SDA_02: track 13.9 -> 90.2 mm
- net I2Cx_SDA_01: track 13.9 -> 88.2 mm
- net I2Cx_SDA_00: track 23.1 -> 82.8 mm
- net I2Cx_SDA_11: track 13.9 -> 71.5 mm
- net I2Cx_SDA_10: track 13.9 -> 63.9 mm
- net I2Cx_SDA_05: track 13.4 -> 60.9 mm, vias 2 -> 4
- net I2Cx_SDA_09: track 13.9 -> 54.8 mm
- net I2Cx_SDA_06: track 13.9 -> 41.2 mm
- net I2Cx_SDA_08: track 13.9 -> 39.6 mm
- net I2Cx_SDA_07: track 13.9 -> 37.9 mm
- net VDD: track 417.8 -> 401.1 mm

Commit message: Finish routing
Connections:
- U4 pad 8: I2Cx_SDA_00 -> I2Cx_SDA_06
- U8 pad 14: I2Cx_SDA_00 -> I2Cx_SDA_04
Routing:
- net I2Cx_SCL: track 322.3 -> 366.0 mm, vias 27 -> 30
- net I2Cx_SDA_06: track 41.2 -> 52.6 mm
- net I2Cx_SDA_04: track 110.4 -> 112.3 mm
- net I2Cx_SDA_05: track 60.9 -> 61.7 mm
- net I2Cx_SDA_01: track 88.2 -> 89.1 mm
- net I2Cx_SDA_10: track 63.9 -> 64.8 mm
- net I2Cx_SDA_07: track 37.9 -> 38.8 mm
- net I2Cx_SDA_09: track 54.8 -> 55.6 mm
- net I2Cx_SDA_03: track 91.6 -> 92.4 mm
- net I2Cx_SDA_00: track 82.8 -> 83.6 mm
- net I2Cx_SDA_02: track 90.2 -> 91.1 mm
- net I2Cx_SDA_11: track 71.5 -> 72.3 mm
- net I2Cx_SDA_08: track 39.6 -> 40.5 mm
- net VDD: track 401.1 -> 400.6 mm, vias 33 -> 32

Commit message: Silkscreen
Parts:
- added G***: LOGO, LOGO, F.Cu at (62.3, 110.7)
- added G***: LOGO, LOGO, F.Cu at (67.2, 110.8)
Routing:
- net I2Cx_SCL: track 366.0 -> 361.1 mm
- net VDD: track 400.6 -> 397.1 mm, vias 32 -> 33
- net I2Cx_SDA_09: track 55.6 -> 59.0 mm
Other:
- board text added: "<24-AuEst"
- board text added: ">"
- board text added: "Rev. 1"
- board text added: "ayu.land/luminography"
